File: LapX.kicad_pcb (KiCad board)
At the start: 2 copper layers, 89 x 63 mm, 83 parts, among them J1 Conn_01x12, J2 Conn_02x01, J3 USB_C_Receptacle_PowerOnly_6P, J4 Micro_SD_Card_Det2, Q1 BSS138, Q2 BSS138, Q3 BSS138, Q4 BSS138, U1 TCMT4100, U2 TCMT4100

Commit message: Layout nearly done
Parts:
- moved C2 2.98 mm to (146.2, 63.2)
- moved C1 2.98 mm to (143.1, 63.2)
- moved C3 1.60 mm to (154.4, 98.6)
- moved RN1 1.48 mm to (148.1, 97.3)
- moved C4 1.35 mm to (154.4, 100.8)
Connections:
- net Net-(D2-A) renamed /VIN_F
- net Net-(FB1-Pad2) renamed /VIN
- J4 pad 11: unconnected-(J4-SHIELD-Pad11) -> GND
- RN1 pad 1: /NU_DAT2 -> /NU_DET1
- RN1 pad 2: /~{CS} -> /NU_DAT2
- RN1 pad 3: /MOSI -> /~{CS}
- RN1 pad 4: /CLK -> /MOSI
- RN2 pad 1: /MISO -> /NU_DAT1
- RN2 pad 2: /NU_DAT1 -> /MISO
- RN2 pad 3: /NU_DET1 -> /CLK
Routing:
- net +3.3V: track 0.00 -> 83.7 mm, vias 0 -> 8
- net /~{CS}: track 0.00 -> 29.8 mm
- net /MOSI: track 0.00 -> 29.1 mm
- net /MISO: track 0.00 -> 26.7 mm
- net /CLK: track 0.00 -> 22.3 mm
- net /NU_DET1: track 0.00 -> 16.4 mm
- net /VDD_OUT: track 0.00 -> 8.54 mm
- net /VSS_OUT: track 0.00 -> 6.82 mm
- net /NU_DAT2: track 0.00 -> 5.78 mm
- net /NU_DAT1: track 0.00 -> 5.67 mm
- net GND: vias 0 -> 23
- added copper zone on B.Cu, net +3.3V
- added copper zone on F.Cu, net +3.3V
- added copper zone on F.Cu, net /VIN
- added copper zone on F.Cu, net /VIN_F
- added copper zone on F.Cu, net VBUS

Commit message: Ärbet
Parts:
- added D1: LED, LED_SMD:LED_0603_1608Metric, F.Cu at (153.0, 65.0)
- added D3: LED, LED_SMD:LED_0603_1608Metric, F.Cu at (149.0, 65.0)
- added D4: LED, LED_SMD:LED_0603_1608Metric, F.Cu at (140.6, 100.2)
- added D5: LED, LED_SMD:LED_0603_1608Metric, F.Cu at (143.4, 100.2)
- added D6: LED, LED_SMD:LED_0603_1608Metric, F.Cu at (146.2, 100.2)
- added D7: LED, LED_SMD:LED_0603_1608Metric, F.Cu at (149.0, 100.2)
- added L10: 1u, Inductor_SMD:L_0805_2012Metric, F.Cu at (138.2, 65.8)
- added R34: 120, Resistor_SMD:R_0603_1608Metric, F.Cu at (153.0, 61.0)
- added R35: 330, Resistor_SMD:R_0603_1608Metric, F.Cu at (149.0, 61.0)
- added R36: 120, Resistor_SMD:R_0603_1608Metric, F.Cu at (140.6, 96.8)
- added R37: 120, Resistor_SMD:R_0603_1608Metric, F.Cu at (143.4, 96.8)
- added R38: 120, Resistor_SMD:R_0603_1608Metric, F.Cu at (146.2, 96.8)
- added R39: 120, Resistor_SMD:R_0603_1608Metric, F.Cu at (149.0, 96.8)
- J1: footprint Connector_PinHeader_2.54mm:PinHeader_1x12_P2.54mm_Vertical -> Connector_PinHeader_2.54mm:PinHeader_1x12_P2.54mm_Horizontal
- J2: footprint Connector_PinHeader_2.54mm:PinHeader_1x02_P2.54mm_Vertical -> Connector_JST:JST_EH_B2B-EH-A_1x02_P2.50mm_Vertical
- J4, R10, R11, R12, R13: moved to B.Cu
- moved J1 28.8 mm to (134.1, 94.4), turned to 180 degrees
- moved RN1 17.6 mm to (165.6, 99.0), turned to -90 degrees
- moved C1 17.5 mm to (160.7, 63.9), turned to -90 degrees
- moved D2 15.4 mm to (164.2, 62.8)
- moved C7 15.2 mm to (167.2, 61.5)
- moved J3 14.6 mm to (162.0, 56.0)
- moved R26 14.3 mm to (139.2, 72.4)
- moved R27 14.2 mm to (139.2, 78.4)
- moved R14 14.1 mm to (139.2, 70.8)
- moved R28 14.1 mm to (139.1, 84.4)
- moved R15 14.0 mm to (139.2, 76.8)
- moved R29 13.9 mm to (139.0, 90.6)
- moved R16 13.9 mm to (139.1, 82.8)
- moved R17 13.7 mm to (139.0, 89.0)
- moved C8 13.5 mm to (141.6, 71.6)
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Connections:
- net /INPUT_OPTO/CHANNEL_1_PICO renamed /CHANNEL_1_PICO
- net /INPUT_OPTO/CHANNEL_2_PICO renamed /CHANNEL_2_PICO
- net /INPUT_OPTO/CHANNEL_3_PICO renamed /CHANNEL_3_PICO
- net /INPUT_OPTO/CHANNEL_4_PICO renamed /CHANNEL_4_PICO
- A1 pad 25: unconnected-(A1-GPIO19-Pad25) -> /DEBUG_LED1
- A1 pad 26: unconnected-(A1-GPIO20-Pad26) -> /DEBUG_LED2
- A1 pad 27: unconnected-(A1-GPIO21-Pad27) -> /DEBUG_LED3
- A1 pad 29: unconnected-(A1-GPIO22-Pad29) -> /DEBUG_LED4
- C21 pad 2: /VSS_OUT -> GND
- J1 pad 1: /RELAIS_1 -> /RELAIS_3
- J1 pad 10: /INPUT_FILTER/CH4_INPUT_N -> /INPUT_FILTER/CH1_INPUT_P
- J1 pad 11: /RELAIS_4 -> /RELAIS_2
- J1 pad 12: /RELAIS_3 -> /RELAIS_1
- J1 pad 2: /RELAIS_2 -> /RELAIS_4
- J1 pad 3: /INPUT_FILTER/CH1_INPUT_P -> /INPUT_FILTER/CH4_INPUT_N
- J1 pad 4: /INPUT_FILTER/CH1_INPUT_N -> /INPUT_FILTER/CH4_INPUT_P
- J1 pad 5: /INPUT_FILTER/CH2_INPUT_P -> /INPUT_FILTER/CH3_INPUT_N
- J1 pad 6: /INPUT_FILTER/CH2_INPUT_N -> /INPUT_FILTER/CH3_INPUT_P
- J1 pad 7: /INPUT_FILTER/CH3_INPUT_P -> /INPUT_FILTER/CH2_INPUT_N
- J1 pad 8: /INPUT_FILTER/CH3_INPUT_N -> /INPUT_FILTER/CH2_INPUT_P
- J1 pad 9: /INPUT_FILTER/CH4_INPUT_P -> /INPUT_FILTER/CH1_INPUT_N
- RN1 pad 1: /NU_DET1 -> /MOSI
- RN1 pad 2: /NU_DAT2 -> /~{CS}
- RN1 pad 3: /~{CS} -> /NU_DAT2
- RN1 pad 4: /MOSI -> /NU_DET1
Routing:
- net +3.3V: track 83.7 -> 0.00 mm, vias 8 -> 0
- net /RELAIS_3: track 63.6 -> 0.00 mm
- net /RELAIS_4: track 60.0 -> 0.00 mm
- net /RELAIS_2: track 39.6 -> 0.00 mm
- net /RELAIS_1: track 39.6 -> 0.00 mm
- net /~{CS}: track 29.8 -> 0.00 mm
- net /MOSI: track 29.1 -> 0.00 mm
- net /CHANNEL_4_PICO: track 28.6 -> 0.00 mm, vias 1 -> 0
- net /CHANNEL_1_PICO: track 28.4 -> 0.00 mm, vias 1 -> 0
- net /CHANNEL_3_PICO: track 27.8 -> 0.00 mm, vias 1 -> 0
- net /CHANNEL_2_PICO: track 27.5 -> 0.00 mm, vias 1 -> 0
- net /MISO: track 26.7 -> 0.00 mm
- net /CLK: track 22.3 -> 0.00 mm
- net /INPUT_FILTER/CH_1_FILT_OUT: track 16.6 -> 0.00 mm, vias 1 -> 0
- net /NU_DET1: track 16.4 -> 0.00 mm
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- removed copper zone on B.Cu, net +3.3V
- removed copper zone on F.Cu, net VBUS
Other:
- board size 89 x 63 mm -> 81.2 x 54.5 mm

Commit message: Layout fast fertig
Parts:
- added G***: LOGO, 00_Graphic_Symbols:ANR_LOGO_F11, B.Cu at (183.9, 73.8)
- J1: footprint Connector_PinHeader_2.54mm:PinHeader_1x12_P2.54mm_Horizontal -> 00_Connector:PHOENIX_1725753
- J2: footprint Connector_JST:JST_EH_B2B-EH-A_1x02_P2.50mm_Vertical -> 00_Connector:PHOENIX_1725656
- J3: footprint Connector_USB:USB_C_Receptacle_HRO_TYPE-C-31-M-17 -> Connector_USB:USB_C_Receptacle_GCT_USB4125-xx-x_6P_TopMnt_Horizontal
- moved J1 29.0 mm to (130.5, 65.5), turned to -90 degrees
- moved RN2 11.9 mm to (166.0, 98.8), turned to 90 degrees
- moved RN1 10.2 mm to (155.4, 99.4), turned to 90 degrees
- moved L10 8.41 mm to (145.8, 62.2), turned to 0 degrees
- moved D3 7.25 mm to (154.6, 60.4), turned to -90 degrees
- moved C4 7.15 mm to (161.2, 100.8), turned to 0 degrees
- moved C21 6.58 mm to (146.8, 64.6), turned to 90 degrees
- moved R35 6.18 mm to (154.6, 63.6)
- moved D4 5.61 mm to (146.2, 100.2)
- moved D6 5.61 mm to (140.6, 100.2)
- moved R36 5.61 mm to (146.2, 96.8), turned to -90 degrees
- moved R38 5.61 mm to (140.6, 96.8), turned to -90 degrees
- moved D5 5.59 mm to (149.0, 100.2)
- moved D7 5.59 mm to (143.4, 100.2)
- moved R37 5.59 mm to (149.0, 96.8), turned to -90 degrees
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Connections:
- J1 pad 1: /RELAIS_3 -> /RELAIS_1
- J1 pad 10: /INPUT_FILTER/CH1_INPUT_P -> /INPUT_FILTER/CH4_INPUT_N
- J1 pad 11: /RELAIS_2 -> /RELAIS_4
- J1 pad 12: /RELAIS_1 -> /RELAIS_3
- J1 pad 2: /RELAIS_4 -> /RELAIS_2
- J1 pad 3: /INPUT_FILTER/CH4_INPUT_N -> /INPUT_FILTER/CH1_INPUT_P
- J1 pad 4: /INPUT_FILTER/CH4_INPUT_P -> /INPUT_FILTER/CH1_INPUT_N
- J1 pad 5: /INPUT_FILTER/CH3_INPUT_N -> /INPUT_FILTER/CH2_INPUT_P
- J1 pad 6: /INPUT_FILTER/CH3_INPUT_P -> /INPUT_FILTER/CH2_INPUT_N
- J1 pad 7: /INPUT_FILTER/CH2_INPUT_N -> /INPUT_FILTER/CH3_INPUT_P
- J1 pad 8: /INPUT_FILTER/CH2_INPUT_P -> /INPUT_FILTER/CH3_INPUT_N
- J1 pad 9: /INPUT_FILTER/CH1_INPUT_N -> /INPUT_FILTER/CH4_INPUT_P
- RN1 pad 1: /MOSI -> /NU_DET1
- RN1 pad 2: /~{CS} -> /NU_DAT2
- RN1 pad 3: /NU_DAT2 -> /~{CS}
- RN1 pad 4: /NU_DET1 -> /MOSI
- RN2 pad 1: /NU_DAT1 -> /CLK
- RN2 pad 3: /CLK -> /NU_DAT1
Routing:
- net +3.3V: track 0.00 -> 155.3 mm, vias 0 -> 9
- net GND: track 0.00 -> 59.0 mm, vias 6 -> 48
- net /DEBUG_LED4: track 0.00 -> 56.4 mm, vias 0 -> 1
- net /DEBUG_LED3: track 0.00 -> 53.3 mm, vias 0 -> 1
- net /DEBUG_LED2: track 0.00 -> 51.4 mm, vias 0 -> 1
- net /RELAIS_3: track 0.00 -> 50.6 mm
- net /DEBUG_LED1: track 0.00 -> 49.8 mm, vias 0 -> 1
- net /RELAIS_4: track 0.00 -> 40.3 mm
- net /CHANNEL_1_PICO: track 0.00 -> 27.5 mm, vias 0 -> 1
- net /RELAIS_2: track 0.00 -> 25.4 mm
- net /RELAIS_1: track 0.00 -> 25.0 mm
- net /CHANNEL_3_PICO: track 0.00 -> 24.8 mm, vias 0 -> 1
- net /CHANNEL_2_PICO: track 0.00 -> 24.7 mm, vias 0 -> 1
- net /MOSI: track 0.00 -> 24.4 mm, vias 0 -> 2
- net /CHANNEL_4_PICO: track 0.00 -> 21.2 mm, vias 0 -> 1
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- added copper zone on F.Cu, net VBUS
Other:
- board text added: "1_N"
- board text added: "1_P"
- board text added: "2_N"
- board text added: "2_P"
- board text added: "3_N"
- board text added: "3_P"
- board text added: "4_N"
- board text added: "4_P"
- board text added: "LapX"
- board text added: "R1"
- board text added: "R2"
- board text added: "R3"
- board text added: "R4"
- board text added: "SENSOR POWER"

Commit message: Layout nearly finished
Parts:
- added G***: LOGO, 00_Graphic_Symbols:USB_Type_C, F.Cu at (169.8, 56.4)
- added G***: LOGO, 00_Graphic_Symbols:RaspberryPie, B.Cu at (183.3, 79.0)
- added REF**: LayerMarker_2_3.81x2.54mm_TextH1mm_P1.27mm_Named_BottomMirr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, Symbol:LayerMarker_2_3.81x2.54mm_TextH1mm_P1.27mm_Named_BottomMirrored, F.Cu at (131.3, 63.4)
- added REF**: ESD-Logo_6.6x6mm_SilkScreen, Symbol:ESD-Logo_6.6x6mm_SilkScreen, B.Cu at (146.6, 97.2)
- added REF**: KiCad-Logo2_5mm_SilkScreen, Symbol:KiCad-Logo2_5mm_SilkScreen, B.Cu at (144.4, 85.8)
- added REF**: WEEE-Logo_4.2x6mm_SilkScreen, Symbol:WEEE-Logo_4.2x6mm_SilkScreen, B.Cu at (139.4, 97.2)
- added REF**: Symbol_Danger_8x8mm_Copper, Symbol:Symbol_Danger_8x8mm_Copper, B.Cu at (183.5, 101.6)
- moved G*** 39.5 mm to (144.5, 76.9), turned to 180 degrees
Other:
- board text added: "Rev 1"
- board text added: "Usable with Raspberry Pi pico"
- board text added: "microSD"
- board text added: "pico"

Commit message: Letzte Changes
Parts:
- added C22: 100n, Capacitor_SMD:C_0603_1608Metric, B.Cu at (183.6, 88.1)
- added C23: 100n, Capacitor_SMD:C_0603_1608Metric, B.Cu at (183.6, 86.5)
- added C24: 100n, Capacitor_SMD:C_0603_1608Metric, B.Cu at (183.6, 84.9)
- added C25: 100n, Capacitor_SMD:C_0603_1608Metric, B.Cu at (183.6, 83.3)
- added C26: 100n, Capacitor_SMD:C_0603_1608Metric, B.Cu at (183.6, 81.7)
- added J5: Conn_01x06_Socket, Connector_PinHeader_2.54mm:PinHeader_1x06_P2.54mm_Vertical, F.Cu at (196.9, 91.5)
- added R40: 330, Resistor_SMD:R_0603_1608Metric, B.Cu at (187.6, 82.0)
- added RN4: 47k, Resistor_SMD:R_Array_Convex_4x0603, B.Cu at (165.2, 82.9)
- added RN5: 330, Resistor_SMD:R_Array_Convex_4x0603, B.Cu at (187.7, 85.5)
- C10, C11, C12, C13, C14, C15, C16, C17, C18, C19, C8, C9: value 100n -> 1u
- C20, C21: value 100n -> 10u
- R14, R15, R16, R17, R26, R27, R28, R29: value 10 -> 1k
- R30, R31, R32, R33: value 1k -> 330
- moved G*** 11.2 mm to (183.2, 67.8)
Connections:
- A1 pad 21: unconnected-(A1-GPIO16-Pad21) -> /DEBUG_LED1
- A1 pad 22: unconnected-(A1-GPIO17-Pad22) -> /DEBUG_LED2
- A1 pad 24: unconnected-(A1-GPIO18-Pad24) -> /DEBUG_LED3
- A1 pad 25: /DEBUG_LED1 -> /DEBUG_LED4
- A1 pad 26: /DEBUG_LED2 -> Net-(A1-GPIO20)
- A1 pad 27: /DEBUG_LED3 -> Net-(A1-GPIO21)
- A1 pad 29: /DEBUG_LED4 -> Net-(A1-GPIO22)
- A1 pad 31: unconnected-(A1-GPIO26_ADC0-Pad31) -> Net-(A1-GPIO26_ADC0)
- A1 pad 32: unconnected-(A1-GPIO27_ADC1-Pad32) -> Net-(A1-GPIO27_ADC1)
- U2 pad 1: /RELAIS_1 -> Net-(R30-Pad1)
- U2 pad 10: Net-(R33-Pad1) -> VBUS
- U2 pad 11: GND -> /RELAIS_3
- U2 pad 12: Net-(R32-Pad1) -> VBUS
- U2 pad 13: GND -> /RELAIS_2
- U2 pad 14: Net-(R31-Pad1) -> VBUS
- U2 pad 15: GND -> /RELAIS_1
- U2 pad 16: Net-(R30-Pad1) -> VBUS
- U2 pad 3: /RELAIS_2 -> Net-(R31-Pad1)
- U2 pad 5: /RELAIS_3 -> Net-(R32-Pad1)
- U2 pad 7: /RELAIS_4 -> Net-(R33-Pad1)
- U2 pad 9: GND -> /RELAIS_4
Routing:
- net VBUS: track 3.76 -> 39.7 mm, vias 0 -> 3
- net Net-(J5-Pin_6): track 0.00 -> 22.8 mm
- net +3.3V: track 155.3 -> 176.2 mm
- net Net-(J5-Pin_5): track 0.00 -> 17.6 mm
- net Net-(J5-Pin_4): track 0.00 -> 17.4 mm
- net /RELAIS_4: track 40.3 -> 57.5 mm, vias 0 -> 2
- net Net-(J5-Pin_3): track 0.00 -> 15.4 mm, vias 0 -> 1
- net Net-(J5-Pin_2): track 0.00 -> 14.9 mm
- net /DEBUG_LED2: track 51.4 -> 59.8 mm
- net Net-(R33-Pad1): track 3.43 -> 11.7 mm
- net GND: track 59.0 -> 66.9 mm, vias 48 -> 63
- net Net-(A1-GPIO20): track 0.00 -> 7.61 mm, vias 0 -> 1
- net Net-(A1-GPIO27_ADC1): track 0.00 -> 7.54 mm
- net /CHANNEL_4_PICO: track 21.2 -> 28.6 mm
- net Net-(R32-Pad1): track 3.31 -> 10.4 mm
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Other:
- board text added: "+3.3V"
- board text added: "+5V"
- board text added: "IN1"
- board text added: "IN2"
- board text added: "IN3"
- board text added: "IN4"
- board text added: "IN5"
- board text removed: "Usable with Raspberry Pi pico"
