File: LapX.kicad_pcb (KiCad board)
At the start: 2 copper layers, 81.2 x 54.5 mm, 113 parts, among them J1 Conn_01x12, J2 Conn_02x01, J3 USB_C_Receptacle_PowerOnly_6P, J4 Micro_SD_Card_Det2, J5 Conn_01x06_Socket, Q1 BSS138, Q2 BSS138, Q3 BSS138, Q4 BSS138, U1 TCMT4100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

Commit message: Small stuff
Routing:
- net GND: vias 63 -> 75
