File: LapX.kicad_sch (KiCad schematic)
At the start: 22 parts, among them J1 Conn_02x05_Top_Bottom, J2 USB_C_Receptacle_PowerOnly_6P, J3 Micro_SD_Card_Det2, J4 Conn_02x01, U1 TCMT4100

Commit message: Ärbet
Parts:
- removed J1: Conn_02x05_Top_Bottom, symbol Connector_Generic:Conn_02x05_Top_Bottom
- removed R3, R4, R5, R6: 1k, symbol Device:R
- removed U1: TCMT4100, Package_SO:SOP-16_4.4x10.4mm_P1.27mm, symbol Isolator:TCMT4100
- added C20, C21: 100n, Capacitor_SMD:C_0603_1608Metric, symbol Device:C
- added H1, H2, H3, H4: MountingHole, MountingHole:MountingHole_3.2mm_M3_DIN965_Pad_TopBottom, symbol Mechanical:MountingHole
- added J1: Conn_01x12, Connector_PinHeader_2.54mm:PinHeader_1x12_P2.54mm_Vertical, symbol Connector_Generic:Conn_01x12
- added L9: 1u, Inductor_SMD:L_0805_2012Metric, symbol Device:L
- added R30, R31, R32, R33: 1k, Resistor_SMD:R_0603_1608Metric, symbol Device:R
- added RN3: 33, Resistor_SMD:R_Array_Convex_4x0603, symbol Device:R_Pack04_Split
- added U2: TCMT4100, Package_SO:SOP-16_4.4x10.4mm_P1.27mm, symbol Isolator:TCMT4100
- A1: footprint Module:RaspberryPi_Pico_Common_Unspecified -> Module:RaspberryPi_Pico_Common_THT
- C1, C2, C3, C5, C6, C7: footprint (none) -> Capacitor_SMD:C_0805_2012Metric
- C4: footprint (none) -> Capacitor_SMD:C_0603_1608Metric
- FB1: footprint (none) -> Inductor_SMD:L_0603_1608Metric
- J2: renamed from J4; footprint (none) -> Connector_PinHeader_2.54mm:PinHeader_1x02_P2.54mm_Vertical
- J3: renamed from J2; footprint (none) -> Connector_USB:USB_C_Receptacle_HRO_TYPE-C-31-M-17
- J4: renamed from J3; footprint (none) -> Connector_Card:microSD_HC_Molex_104031-0811
- R1: footprint (none) -> Resistor_SMD:R_0603_1608Metric
- RN1, RN2: value 4k7 -> 47k; footprint (none) -> Resistor_SMD:R_Array_Convex_4x0603
Connections:
- net +3.3V: now also RN1.5 (R4.2), RN1.6 (R3.2), RN1.7 (R2.2), RN1.8 (R1.2), RN2.6 (R3.2), RN2.7 (R2.2), RN2.8 (R1.2)
- net CLK: now also RN1.4 (R4.1), RN3.1 (R1.1)
- net GND: now also U2.11, U2.13, U2.15, U2.2, U2.4, U2.6, U2.8, U2.9
- net MISO: now also RN2.1 (R1.1), RN3.3 (R3.1)
- net MOSI: now also RN1.3 (R3.1), RN3.2 (R2.1)
- net NU_DAT1: now also RN2.2 (R2.1)
- net NU_DAT2: now also RN1.1 (R1.1)
- net NU_DET1: now also RN2.3 (R3.1)
- net VBUS: now also C21.1, L9.2
- net ~{CS}: now also RN1.2 (R2.1), RN3.4 (R4.1)
- net VSS_OUT: now reaches J2.1 (Pin_1)
- net VSS_OUT: now also C20.2, C21.2
- net VDD_OUT: now reaches J2.2 (Pin_2)
- net VDD_OUT: now also C20.1, L9.1
- net CLK_R: now reaches A1.14 (GPIO10)
- net CLK_R: now also RN3.8 (R1.2)
- net MOSI_R: now reaches A1.15 (GPIO11)
- net MOSI_R: now also RN3.7 (R2.2)
- net MISO_R: now reaches A1.16 (GPIO12)
- net MISO_R: now also RN3.6 (R3.2)
- net ~{CS_R}: now reaches A1.17 (GPIO13)
- net ~{CS_R}: now also RN3.5 (R4.2)
- net GPIO_2: now reaches A1.4 (GPIO2)
- net GPIO_2: now also R30.2
- net GPIO_3: now reaches A1.5 (GPIO3)
- net GPIO_3: now also R31.2
- net GPIO_4: now reaches A1.6 (GPIO4)
- net GPIO_4: now also R32.2
- net GPIO_5: now reaches A1.7 (GPIO5)
- net GPIO_5: now also R33.2
- net CHANNEL_1_IN renamed INPUT_OPTO/CHANNEL_1_PICO
- net CHANNEL_2_IN renamed INPUT_OPTO/CHANNEL_2_PICO
- net CHANNEL_3_IN renamed INPUT_OPTO/CHANNEL_3_PICO
- net CHANNEL_4_IN renamed INPUT_OPTO/CHANNEL_4_PICO
- new net: R33.1, U2.10
- new net: R32.1, U2.12
- new net: R30.1, U2.16
- new net: R31.1, U2.14
- new net INPUT_FILTER/CH1_INPUT_N: J1.4 (Pin_4)
- new net INPUT_FILTER/CH1_INPUT_P: J1.3 (Pin_3)
- new net INPUT_FILTER/CH2_INPUT_N: J1.6 (Pin_6)
- new net INPUT_FILTER/CH2_INPUT_P: J1.5 (Pin_5)
- new net INPUT_FILTER/CH3_INPUT_N: J1.8 (Pin_8)
- new net INPUT_FILTER/CH3_INPUT_P: J1.7 (Pin_7)
- new net INPUT_FILTER/CH4_INPUT_N: J1.10 (Pin_10)
- new net INPUT_FILTER/CH4_INPUT_P: J1.9 (Pin_9)
- new net RELAIS_1: J1.1 (Pin_1), U2.1
- new net RELAIS_2: J1.2 (Pin_2), U2.3
- new net RELAIS_3: J1.12 (Pin_12), U2.5
- new net RELAIS_4: J1.11 (Pin_11), U2.7
- no-connect marks 0 -> 20
Other:
- added sheet INPUT_FILTER (input_filter.kicad_sch)
- added sheet INPUT_OPTO (Input_Opto.kicad_sch)
- added sheet Input_FET (Input_fet.kicad_sch)
- moved on the sheet: A1, C1, C2, C5, C6, C7, D2, FB1, J2, J3, R1, RN1A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

Commit message: Layout nearly done
Connections:
- net CLK: now also RN2.3 (R3.1); no longer RN1.4 (R4.1)
- net GND: now also J4.11 (SHIELD)
- net MISO: now also RN2.2 (R2.1); no longer RN2.1 (R1.1)
- net MOSI: now also RN1.4 (R4.1); no longer RN1.3 (R3.1)
- net NU_DAT1: now also RN2.1 (R1.1); no longer RN2.2 (R2.1)
- net NU_DAT2: now also RN1.2 (R2.1); no longer RN1.1 (R1.1)
- net NU_DET1: now also RN1.1 (R1.1); no longer RN2.3 (R3.1)
- net ~{CS}: now also RN1.3 (R3.1); no longer RN1.2 (R2.1)
- net VIN_F: now reaches C7.1, D2.2 (A), FB1.1
- net VIN: now reaches FB1.2, J3.A9 (VBUS), J3.B9 (VBUS)
Other:
- moved on the sheet: FB1, RN1A, RN1B, RN1C, RN1D, RN2A, RN2B, RN2C, RN2D

Commit message: Ärbet
Parts:
- added D1, D3, D4, D5, D6, D7: LED, LED_SMD:LED_0603_1608Metric, symbol Device:LED
- added L10: 1u, Inductor_SMD:L_0805_2012Metric, symbol Device:L
- added R34, R36, R37, R38, R39: 120, Resistor_SMD:R_0603_1608Metric, symbol Device:R
- added R35: 330, Resistor_SMD:R_0603_1608Metric, symbol Device:R
- J1: footprint Connector_PinHeader_2.54mm:PinHeader_1x12_P2.54mm_Vertical -> Connector_PinHeader_2.54mm:PinHeader_1x12_P2.54mm_Horizontal
- J2: footprint Connector_PinHeader_2.54mm:PinHeader_1x02_P2.54mm_Vertical -> Connector_JST:JST_EH_B2B-EH-A_1x02_P2.50mm_Vertical
Connections:
- net +3.3V: now also R34.1
- net GND: now also C21.2, D1.1 (K), D3.1 (K), D4.1 (K), D5.1 (K), D6.1 (K), D7.1 (K), L10.2
- net INPUT_FILTER/CH1_INPUT_N: now also J1.9 (Pin_9); no longer J1.4 (Pin_4)
- net INPUT_FILTER/CH1_INPUT_P: now also J1.10 (Pin_10); no longer J1.3 (Pin_3)
- net INPUT_FILTER/CH2_INPUT_N: now also J1.7 (Pin_7); no longer J1.6 (Pin_6)
- net INPUT_FILTER/CH2_INPUT_P: now also J1.8 (Pin_8); no longer J1.5 (Pin_5)
- net INPUT_FILTER/CH3_INPUT_N: now also J1.5 (Pin_5); no longer J1.8 (Pin_8)
- net INPUT_FILTER/CH3_INPUT_P: now also J1.6 (Pin_6); no longer J1.7 (Pin_7)
- net INPUT_FILTER/CH4_INPUT_N: now also J1.3 (Pin_3); no longer J1.10 (Pin_10)
- net INPUT_FILTER/CH4_INPUT_P: now also J1.4 (Pin_4); no longer J1.9 (Pin_9)
- net MOSI: now also RN1.1 (R1.1); no longer RN1.4 (R4.1)
- net NU_DAT2: now also RN1.3 (R3.1); no longer RN1.2 (R2.1)
- net NU_DET1: now also RN1.4 (R4.1); no longer RN1.1 (R1.1)
- net RELAIS_1: now also J1.12 (Pin_12); no longer J1.1 (Pin_1)
- net RELAIS_2: now also J1.11 (Pin_11); no longer J1.2 (Pin_2)
- net RELAIS_3: now also J1.1 (Pin_1); no longer J1.12 (Pin_12)
- net RELAIS_4: now also J1.2 (Pin_2); no longer J1.11 (Pin_11)
- net VBUS: now also R35.1
- net VSS_OUT: now also L10.1; no longer C21.2
- net ~{CS}: now also RN1.2 (R2.1); no longer RN1.3 (R3.1)
- net DEBUG_LED1: now reaches A1.25 (GPIO19)
- net DEBUG_LED1: now also R37.1
- net DEBUG_LED2: now reaches A1.26 (GPIO20)
- net DEBUG_LED2: now also R36.1
- net DEBUG_LED3: now reaches A1.27 (GPIO21)
- net DEBUG_LED3: now also R39.1
- net DEBUG_LED4: now reaches A1.29 (GPIO22)
- net DEBUG_LED4: now also R38.1
- net INPUT_OPTO/CHANNEL_1_PICO renamed CHANNEL_1_PICO
- net INPUT_OPTO/CHANNEL_2_PICO renamed CHANNEL_2_PICO
- net INPUT_OPTO/CHANNEL_3_PICO renamed CHANNEL_3_PICO
- net INPUT_OPTO/CHANNEL_4_PICO renamed CHANNEL_4_PICO
- new net: D1.2 (A), R34.2
- new net: D7.2 (A), R39.2
- new net: D6.2 (A), R38.2
- new net: D4.2 (A), R36.2
- new net: D5.2 (A), R37.2
- new net: D3.2 (A), R35.2
- no-connect marks 20 -> 16
Other:
- moved on the sheet: J1, RN1A, RN1B, RN1C, RN1D

Commit message: Layout fast fertig
Parts:
- J1: footprint Connector_PinHeader_2.54mm:PinHeader_1x12_P2.54mm_Horizontal -> 00_Connector:PHOENIX_1725753
- J2: footprint Connector_JST:JST_EH_B2B-EH-A_1x02_P2.50mm_Vertical -> 00_Connector:PHOENIX_1725656
- J3: footprint Connector_USB:USB_C_Receptacle_HRO_TYPE-C-31-M-17 -> Connector_USB:USB_C_Receptacle_GCT_USB4125-xx-x_6P_TopMnt_Horizontal
Connections:
- net CLK: now also RN2.1 (R1.1); no longer RN2.3 (R3.1)
- net INPUT_FILTER/CH1_INPUT_N: now also J1.4 (Pin_4); no longer J1.9 (Pin_9)
- net INPUT_FILTER/CH1_INPUT_P: now also J1.3 (Pin_3); no longer J1.10 (Pin_10)
- net INPUT_FILTER/CH2_INPUT_N: now also J1.6 (Pin_6); no longer J1.7 (Pin_7)
- net INPUT_FILTER/CH2_INPUT_P: now also J1.5 (Pin_5); no longer J1.8 (Pin_8)
- net INPUT_FILTER/CH3_INPUT_N: now also J1.8 (Pin_8); no longer J1.5 (Pin_5)
- net INPUT_FILTER/CH3_INPUT_P: now also J1.7 (Pin_7); no longer J1.6 (Pin_6)
- net INPUT_FILTER/CH4_INPUT_N: now also J1.10 (Pin_10); no longer J1.3 (Pin_3)
- net INPUT_FILTER/CH4_INPUT_P: now also J1.9 (Pin_9); no longer J1.4 (Pin_4)
- net MOSI: now also RN1.4 (R4.1); no longer RN1.1 (R1.1)
- net NU_DAT1: now also RN2.3 (R3.1); no longer RN2.1 (R1.1)
- net NU_DAT2: now also RN1.2 (R2.1); no longer RN1.3 (R3.1)
- net NU_DET1: now also RN1.1 (R1.1); no longer RN1.4 (R4.1)
- net RELAIS_1: now also J1.1 (Pin_1); no longer J1.12 (Pin_12)
- net RELAIS_2: now also J1.2 (Pin_2); no longer J1.11 (Pin_11)
- net RELAIS_3: now also J1.12 (Pin_12); no longer J1.1 (Pin_1)
- net RELAIS_4: now also J1.11 (Pin_11); no longer J1.2 (Pin_2)
- net ~{CS}: now also RN1.3 (R3.1); no longer RN1.2 (R2.1)
- no-connect marks 16 -> 18
Other:
- moved on the sheet: J1
Changed lines of the file:
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@@
 	)
 	(no_connect
+		(at 247.65 96.52)
+	)
+	(no_connect
 		(at 293.37 106.68)
 	)
@@
 	)
 	(no_connect
+		(at 247.65 93.98)
+	)
+	(no_connect
 		(at 247.65 104.14)
 	)
@@
 	(wire
 		(pts
+			(xy 217.17 242.57) (xy 217.17 232.41)
+		)
+		(stroke
+			(width 0)
+			(type default)
+		)
+	)
+	(wire
+		(pts
 			(xy 88.9 217.17) (xy 105.41 217.17)
 		)
@@
 	(wire
 		(pts
-			(xy 207.01 242.57) (xy 207.01 232.41)
-		)
-		(stroke
-			(width 0)
-			(type default)
-		)
-	)
-	(wire
-		(pts
 			(xy 241.3 173.99) (xy 252.73 173.99)
 		)
@@
 	(wire
 		(pts
-			(xy 196.85 242.57) (xy 196.85 232.41)
-		)
-		(stroke
-			(width 0)
-			(type default)
-		)
-	)
-	(wire
-		(pts
 			(xy 275.59 74.93) (xy 275.59 78.74)
 		)
@@
 	(wire
 		(pts
-			(xy 217.17 242.57) (xy 217.17 232.41)
+			(xy 48.26 138.43) (xy 48.26 128.27)
 		)
 		(stroke
@@
 	(wire
 		(pts
-			(xy 48.26 138.43) (xy 48.26 128.27)
+			(xy 130.81 201.93) (xy 120.65 201.93)
 		)
 		(stroke
@@
 	(wire
 		(pts
-			(xy 130.81 201.93) (xy 120.65 201.93)
+			(xy 278.13 50.8) (xy 278.13 53.34)
 		)
 		(stroke
@@
 	(wire
 		(pts
-			(xy 278.13 50.8) (xy 278.13 53.34)
+			(xy 130.81 217.17) (xy 120.65 217.17)
 		)
 		(stroke
@@
 	(wire
 		(pts
-			(xy 130.81 217.17) (xy 120.65 217.17)
+			(xy 335.28 40.64) (xy 345.44 40.64)
 		)
 		(stroke
@@
 	(wire
 		(pts
-			(xy 335.28 40.64) (xy 345.44 40.64)
+			(xy 227.33 242.57) (xy 227.33 232.41)
 		)
 		(stroke
@@
 	(wire
 		(pts
+			(xy 247.65 242.57) (xy 247.65 232.41)
+		)
+		(stroke
+			(width 0)
+			(type default)
+		)
+	)
+	(wire
+		(pts
 			(xy 93.98 140.97) (xy 127 140.97)
 		)
@@
 	(wire
 		(pts
-			(xy 217.17 119.38) (xy 217.17 102.87)
+			(xy 257.81 242.57) (xy 257.81 232.41)
 		)
 		(stroke
@@
 	(wire
 		(pts
-			(xy 204.47 121.92) (xy 204.47 124.46)
+			(xy 217.17 119.38) (xy 217.17 102.87)
 		)
 		(stroke
@@
 	(wire
 		(pts
-			(xy 369.57 153.67) (xy 369.57 158.75)
+			(xy 204.47 121.92) (xy 204.47 124.46)
 		)
 		(stroke
@@
 	(wire
 		(pts
-			(xy 307.34 151.13) (xy 381 151.13)
+			(xy 369.57 153.67) (xy 369.57 158.75)
 		)
 		(stroke
@@
 	(wire
 		(pts
-			(xy 392.43 166.37) (xy 392.43 168.91)
+			(xy 307.34 151.13) (xy 381 151.13)
 		)
 		(stroke
@@
 	(wire
 		(pts
-			(xy 247.65 242.57) (xy 247.65 232.41)
+			(xy 392.43 166.37) (xy 392.43 168.91)
 		)
 		(stroke
@@
 	(wire
 		(pts
-			(xy 257.81 242.57) (xy 257.81 232.41)
+			(xy 45.72 113.03) (xy 45.72 100.33)
 		)
 		(stroke
@@
 	(wire
 		(pts
-			(xy 45.72 113.03) (xy 45.72 100.33)
+			(xy 127 179.07) (xy 127 140.97)
 		)
 		(stroke
@@
 	(wire
 		(pts
-			(xy 127 179.07) (xy 127 140.97)
+			(xy 341.63 224.79) (xy 344.17 224.79)
 		)
 		(stroke
@@
 	(wire
 		(pts
-			(xy 341.63 224.79) (xy 344.17 224.79)
+			(xy 207.01 242.57) (xy 207.01 232.41)
 		)
 		(stroke
@@
 	(wire
 		(pts
+			(xy 196.85 242.57) (xy 196.85 232.41)
+		)
+		(stroke
+			(width 0)
+			(type default)
+		)
+	)
+	(wire
+		(pts
 			(xy 97.79 48.26) (xy 90.17 48.26)
 		)
@@
 	(wire
 		(pts
-			(xy 227.33 242.57) (xy 227.33 232.41)
-		)
-		(stroke
-			(width 0)
-			(type default)
-		)
-	)
-	(wire
-		(pts
 			(xy 238.76 134.62) (xy 247.65 134.62)
 		)
@@
 	(wire
 		(pts
-			(xy 237.49 242.57) (xy 237.49 232.41)
-		)
-		(stroke
-			(width 0)
-			(type default)
-		)
-	)
-	(wire
-		(pts
 			(xy 160.02 44.45) (xy 160.02 46.99)
 		)
@@
 	(wire
 		(pts
+			(xy 237.49 242.57) (xy 237.49 232.41)
+		)
+		(stroke
+			(width 0)
+			(type default)
+		)
+	)
+	(wire
+		(pts
 			(xy 175.26 57.15) (xy 175.26 54.61)
 		)
@@
 		)
 	)
-	(label "~{CS}"
-		(at 217.17 242.57 90)
+	(label "MISO"
+		(at 247.65 242.57 90)
 		(effects
 			(font
@@
 		)
 	)
-	(label "MOSI"
-		(at 227.33 242.57 90)
-		(effects
-			(font
-				(size 1.27 1.27)
-			)
-			(justify left bottom)
-		)
-	)
 	(label "RELAIS_4"
 		(at 38.1 133.35 180)
@@
 		)
 	)
-	(label "NU_DAT2"
-		(at 207.01 242.57 90)
-		(effects
-			(font
-				(size 1.27 1.27)
-			)
-			(justify left bottom)
-		)
-	)
 	(label "VIN_F"
 		(at 317.5 40.64 0)
@@
 		)
 	)
-	(label "NU_DET1"
-		(at 196.85 242.57 90)
+	(label "MOSI_R"
+		(at 241.3 173.99 0)
 		(effects
 			(font
@@
 		)
 	)
-	(label "MOSI_R"
-		(at 241.3 173.99 0)
+	(label "CHANNEL_3_PICO"
+		(at 227.33 121.92 0)
 		(effects
 			(font
@@
 		)
 	)
-	(label "CHANNEL_3_PICO"
-		(at 227.33 121.92 0)
+	(label "NU_DAT2"
+		(at 217.17 242.57 90)
 		(effects
 			(font
@@
 		)
 	)
+	(label "~{CS}"
+		(at 207.01 242.57 90)
+		(effects
+			(font
+				(size 1.27 1.27)
+			)
+			(justify left bottom)
+		)
+	)
 	(label "RELAIS_3"
 		(at 38.1 135.89 180)
@@
 		)
 	)
-	(label "MISO"
-		(at 247.65 242.57 90)
+	(label "~{CS_R}"
+		(at 241.3 184.15 0)
 		(effects
 			(font
@@
 		)
 	)
-	(label "~{CS_R}"
-		(at 241.3 184.15 0)
+	(label "NU_DAT1"
+		(at 257.81 242.57 90)
 		(effects
 			(font
@@
 		)
 	)
+	(label "CLK"
+		(at 237.49 242.57 90)
+		(effects
+			(font
+				(size 1.27 1.27)
+			)
+			(justify left bottom)
+		)
+	)
 	(label "DEBUG_LED4"
 		(at 326.39 156.21 0)
@@
 	)
 	(label "MOSI"
-		(at 269.24 173.99 180)
+		(at 196.85 242.57 90)
 		(effects
 			(font
 				(size 1.27 1.27)
 			)
-			(justify right bottom)
+			(justify left bottom)
 		)
 	)
-	(label "MISO"
-		(at 318.77 227.33 0)
+	(label "MOSI"
+		(at 269.24 173.99 180)
 		(effects
 			(font
 				(size 1.27 1.27)
 			)
-			(justify left bottom)
+			(justify right bottom)
 		)
 	)
-	(label "GPIO_5"
-		(at 238.76 114.3 0)
+	(label "MISO"
+		(at 318.77 227.33 0)
 		(effects
 			(font
@@
 		)
 	)
-	(label "NU_DAT1"
-		(at 237.49 242.57 90)
+	(label "NU_DET1"
+		(at 227.33 242.57 90)
 		(effects
 			(font
@@
 		)
 	)
-	(label "CLK"
-		(at 257.81 242.57 90)
+	(label "GPIO_5"
+		(at 238.76 114.3 0)
 		(effects
 			(font
@@
 	(symbol
 		(lib_id "Connector_Generic:Conn_01x12")
-		(at 22.86 123.19 180)
+		(at 22.86 120.65 0)
+		(mirror y)
 		(unit 1)
 		(exclude_from_sim no)
@@
 		(dnp no)
 		(property "Reference" "J1"
-			(at 22.86 142.494 0)
+			(at 22.86 101.346 0)
 			(effects
 				(font
@@
 		)
 		(property "Value" "Conn_01x12"
-			(at 22.86 139.954 0)
+			(at 22.86 103.886 0)
 			(effects
 				(font
@@
 			)
 		)
-		(property "Footprint" "Connector_PinHeader_2.54mm:PinHeader_1x12_P2.54mm_Horizontal"
-			(at 22.86 123.19 0)
+		(property "Footprint" "00_Connector:PHOENIX_1725753"
+			(at 22.86 120.65 0)
 			(effects
 				(font
@@
 		)
 		(property "Datasheet" "~"
-			(at 22.86 123.19 0)
+			(at 22.86 120.65 0)
 			(effects
 				(font
@@
 		)
 		(property "Description" "Generic connector, single row, 01x12, script generated (kicad-library-utils/schlib/autogen/connector/)"
-			(at 22.86 123.19 0)
+			(at 22.86 120.65 0)
 			(effects
 				(font
@@
 		)
 		(property "LCSC" ""
-			(at 22.86 123.19 0)
+			(at 22.86 120.65 0)
 			(effects
 				(font
@@
 			)
 		)
-		(property "Footprint" "Connector_USB:USB_C_Receptacle_HRO_TYPE-C-31-M-17"
+		(property "Footprint" "Connector_USB:USB_C_Receptacle_GCT_USB4125-xx-x_6P_TopMnt_Horizontal"
 			(at 356.87 45.72 0)
 			(effects
@@
 			)
 		)
-		(property "Footprint" "Connector_JST:JST_EH_B2B-EH-A_1x02_P2.50mm_Vertical"
+		(property "Footprint" "00_Connector:PHOENIX_1725656"
 			(at 54.61 34.29 0)
 			(effects

Commit message: Layout nearly finished
Parts:
- C20, C21: value 100n -> 10u
Other:
- note added: "+3.3V LED"
- note added: "+5V LED"
- note added: "Debugging LEDs"
- note added: "GND"
- note added: "INPUT Filter"
- note added: "INPUT with FETs"
- note added: "INPUT with Optocoupler"
- note added: "Iout_max = 750 mA"
- note added: "Micro SD Card for Raspberry Pi pico"
- note added: "OUT"
- note added: "Relais over Optocoupler"
- note added: "Sternpunkt GND an der Lichtschranke"
- note added: "Sternpunkt Stromversorgung am Stecker J2"
- note added: "USB C Power in 5V 1A"
- note added: "VCC"
- moved on the sheet: C20, C21, C3, C4, J1, J2, J4, L10, L9, R30, R31, R32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

Commit message: Letzte Changes
Parts:
- added C22, C23, C24, C25, C26: 100n, Capacitor_SMD:C_0603_1608Metric, symbol Device:C
- added J5: Conn_01x06_Socket, Connector_PinHeader_2.54mm:PinHeader_1x06_P2.54mm_Vertical, symbol Connector:Conn_01x06_Socket
- added R40: 330, Resistor_SMD:R_0603_1608Metric, symbol Device:R
- added RN5: 330, Resistor_SMD:R_Array_Convex_4x0603, symbol Device:R_Pack04_Split
- R30, R31, R32, R33: value 1k -> 330
Connections:
- net +3.3V: now also J5.1 (Pin_1)
- net DEBUG_LED1: now also A1.21 (GPIO16); no longer A1.25 (GPIO19)
- net DEBUG_LED2: now also A1.22 (GPIO17); no longer A1.26 (GPIO20)
- net DEBUG_LED3: now also A1.24 (GPIO18); no longer A1.27 (GPIO21)
- net DEBUG_LED4: now also A1.25 (GPIO19); no longer A1.29 (GPIO22)
- net GND: now also C22.1, C23.1, C24.1, C25.1, C26.1; no longer U2.11, U2.13, U2.15, U2.9
- net RELAIS_1: now also U2.15; no longer U2.1
- net RELAIS_2: now also U2.13; no longer U2.3
- net RELAIS_3: now also U2.11; no longer U2.5
- net RELAIS_4: now also U2.9; no longer U2.7
- net VBUS: now also U2.10, U2.12, U2.14, U2.16
- net at R33.1: now also U2.7; no longer U2.10
- net at R32.1: now also U2.5; no longer U2.12
- net at R30.1: now also U2.1; no longer U2.16
- net at R31.1: now also U2.3; no longer U2.14
- net at A1.31 (GPIO26_ADC0): now also RN5.5 (R4.2)
- net at A1.32 (GPIO27_ADC1): now also R40.1
- new net: C22.2, J5.2 (Pin_2), RN5.1 (R1.1)
- new net: A1.26 (GPIO20), RN5.8 (R1.2)
- new net: C24.2, J5.4 (Pin_4), RN5.3 (R3.1)
- new net: A1.29 (GPIO22), RN5.6 (R3.2)
- new net: C23.2, J5.3 (Pin_3), RN5.2 (R2.1)
- new net: A1.27 (GPIO21), RN5.7 (R2.2)
- new net: C25.2, J5.5 (Pin_5), RN5.4 (R4.1)
- new net: C26.2, J5.6 (Pin_6), R40.2
- no-connect marks 18 -> 13
Other:
- note added: "Debouncing"
- note added: "Notaus Taster Input"
- moved on the sheet: C3, C4, J4, R30, R31, R32, R33, RN1A, RN1B, RN1C, RN1D, RN2A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
