File: input_filter.kicad_sch (KiCad schematic)
At the start: 36 parts

Commit message: Layout nearly finished
Parts:
- R14, R15, R16, R17, R26, R27, R28, R29: value 10 -> 1k
Changed lines of the file:
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@@
 			)
 		)
-		(property "Value" "10"
+		(property "Value" "1k"
 			(at 73.66 101.6 90)
 			(effects
@@
 			)
 		)
-		(property "Value" "10"
+		(property "Value" "1k"
 			(at 73.66 74.93 90)
 			(effects
@@
 			)
 		)
-		(property "Value" "10"
+		(property "Value" "1k"
 			(at 73.66 62.23 90)
 			(effects
@@
 			)
 		)
-		(property "Value" "10"
+		(property "Value" "1k"
 			(at 73.66 142.24 90)
 			(effects
@@
 			)
 		)
-		(property "Value" "10"
+		(property "Value" "1k"
 			(at 73.66 128.27 90)
 			(effects
@@
 			)
 		)
-		(property "Value" "10"
+		(property "Value" "1k"
 			(at 73.66 115.57 90)
 			(effects
@@
 			)
 		)
-		(property "Value" "10"
+		(property "Value" "1k"
 			(at 73.66 154.94 90)
 			(effects
@@
 			)
 		)
-		(property "Value" "10"
+		(property "Value" "1k"
 			(at 73.66 88.9 90)
 			(effects

Commit message: Letzte Changes
Parts:
- C10, C11, C12, C13, C14, C15, C8, C9: value 100n -> 1u
- C16, C17, C18, C19: value 100n -> 1u; now fitted
Changed lines of the file:
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@@
 			)
 		)
-		(property "Value" "100n"
+		(property "Value" "1u"
 			(at 88.9 123.1899 0)
 			(effects
@@
 			)
 		)
-		(property "Value" "100n"
+		(property "Value" "1u"
 			(at 88.9 69.8499 0)
 			(effects
@@
 		(in_bom yes)
 		(on_board yes)
-		(dnp yes)
+		(dnp no)
 		(fields_autoplaced yes)
 		(property "Reference" "C17"
@@
 			)
 		)
-		(property "Value" "100n"
+		(property "Value" "1u"
 			(at 156.21 96.5199 0)
 			(effects
@@
 			)
 		)
-		(property "Value" "100n"
+		(property "Value" "1u"
 			(at 133.35 96.5199 0)
 			(effects
@@
 		(in_bom yes)
 		(on_board yes)
-		(dnp yes)
+		(dnp no)
 		(fields_autoplaced yes)
 		(property "Reference" "C18"
@@
 			)
 		)
-		(property "Value" "100n"
+		(property "Value" "1u"
 			(at 156.21 123.1899 0)
 			(effects
@@
 			)
 		)
-		(property "Value" "100n"
+		(property "Value" "1u"
 			(at 133.35 69.8499 0)
 			(effects
@@
 			)
 		)
-		(property "Value" "100n"
+		(property "Value" "1u"
 			(at 88.9 149.8599 0)
 			(effects
@@
 			)
 		)
-		(property "Value" "100n"
+		(property "Value" "1u"
 			(at 133.35 149.8599 0)
 			(effects
@@
 			)
 		)
-		(property "Value" "100n"
+		(property "Value" "1u"
 			(at 88.9 96.5199 0)
 			(effects
@@
 		(in_bom yes)
 		(on_board yes)
-		(dnp yes)
+		(dnp no)
 		(fields_autoplaced yes)
 		(property "Reference" "C16"
@@
 			)
 		)
-		(property "Value" "100n"
+		(property "Value" "1u"
 			(at 156.21 69.8499 0)
 			(effects
@@
 		(in_bom yes)
 		(on_board yes)
-		(dnp yes)
+		(dnp no)
 		(fields_autoplaced yes)
 		(property "Reference" "C19"
@@
 			)
 		)
-		(property "Value" "100n"
+		(property "Value" "1u"
 			(at 156.21 149.8599 0)
 			(effects
@@
 			)
 		)
-		(property "Value" "100n"
+		(property "Value" "1u"
 			(at 133.35 123.1899 0)
 			(effects
